File: msp-debugger/msp-debugger.kicad_sch (KiCad schematic)
At the start: 23 parts, among them J1 USB_B_Micro, J2 Conn_02x10, SW1 222ADVBA, SW2 222ADVBA, SW3 222ADVBA, SW4 222ADVBA, SW5 222ADVBA, SW6 222ADVBA, U1 ESP32-S2-SOLO, U2 NHD-0420H1Z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

Commit message: finalized pcb
Parts:
- renumbered SW4 to DOWN1, SW5 to ESP_ENABLE1, SW6 to ESP_PROGRAM1, SW2 to RETURN1, SW1 to SET1, SW3 to UP1
Changed lines of the file:
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@@
   (symbol (lib_id "Switch:SW_MEC_5E") (at 172.5168 40.9956 0) (unit 1)
     (in_bom yes) (on_board yes) (dnp no) (fields_autoplaced)
-    (property "Reference" "SW6" (at 172.5168 31.75 0)
+    (property "Reference" "ESP_PROGRAM1" (at 172.5168 31.75 0)
       (effects (font (size 1.27 1.27)))
     )
@@
       (project "msp-debugger"
         (path "/045ba461-bcb4-4373-9dc5-687bfd2826ef"
-          (reference "SW6") (unit 1)
+          (reference "ESP_PROGRAM1") (unit 1)
         )
       )
@@
   (symbol (lib_id "Switch:SW_MEC_5E") (at 137.2108 40.9956 0) (unit 1)
     (in_bom yes) (on_board yes) (dnp no) (fields_autoplaced)
-    (property "Reference" "SW5" (at 137.2108 31.75 0)
+    (property "Reference" "ESP_ENABLE1" (at 137.2108 31.75 0)
       (effects (font (size 1.27 1.27)))
     )
@@
       (project "msp-debugger"
         (path "/045ba461-bcb4-4373-9dc5-687bfd2826ef"
-          (reference "SW5") (unit 1)
+          (reference "ESP_ENABLE1") (unit 1)
         )
       )
@@
   (symbol (lib_id "Switch:SW_MEC_5E") (at 183.1086 103.632 0) (unit 1)
     (in_bom yes) (on_board yes) (dnp no) (fields_autoplaced)
-    (property "Reference" "SW3" (at 183.1086 93.98 0)
+    (property "Reference" "UP1" (at 183.1086 93.98 0)
       (effects (font (size 1.27 1.27)))
     )
@@
       (project "msp-debugger"
         (path "/045ba461-bcb4-4373-9dc5-687bfd2826ef"
-          (reference "SW3") (unit 1)
+          (reference "UP1") (unit 1)
         )
       )
@@
   (symbol (lib_id "Switch:SW_MEC_5E") (at 183.2356 82.677 0) (unit 1)
     (in_bom yes) (on_board yes) (dnp no) (fields_autoplaced)
-    (property "Reference" "SW1" (at 183.2356 73.66 0)
+    (property "Reference" "SET1" (at 183.2356 73.66 0)
       (effects (font (size 1.27 1.27)))
     )
@@
       (project "msp-debugger"
         (path "/045ba461-bcb4-4373-9dc5-687bfd2826ef"
-          (reference "SW1") (unit 1)
+          (reference "SET1") (unit 1)
         )
       )
@@
   (symbol (lib_id "Switch:SW_MEC_5E") (at 183.2356 92.964 0) (unit 1)
     (in_bom yes) (on_board yes) (dnp no) (fields_autoplaced)
-    (property "Reference" "SW2" (at 183.2356 83.82 0)
+    (property "Reference" "RETURN1" (at 183.2356 83.82 0)
       (effects (font (size 1.27 1.27)))
     )
@@
       (project "msp-debugger"
         (path "/045ba461-bcb4-4373-9dc5-687bfd2826ef"
-          (reference "SW2") (unit 1)
+          (reference "RETURN1") (unit 1)
         )
       )
@@
   (symbol (lib_id "Switch:SW_MEC_5E") (at 183.1086 114.554 0) (unit 1)
     (in_bom yes) (on_board yes) (dnp no) (fields_autoplaced)
-    (property "Reference" "SW4" (at 183.1086 105.41 0)
+    (property "Reference" "DOWN1" (at 183.1086 105.41 0)
       (effects (font (size 1.27 1.27)))
     )
@@
       (project "msp-debugger"
         (path "/045ba461-bcb4-4373-9dc5-687bfd2826ef"
-          (reference "SW4") (unit 1)
-        )
-      )
+          (reference "DOWN1") (unit 1)
+        )
+      )
